Commit message: update

File: src/renderer/public/urdf/GRMini1T1_raw.urdf (robot description, URDF)
Before this commit: robot GRMini1T1, 29 links, 28 joints
Links:
- link base_link: geometry collision mesh filename=../meshes/base_link.STL; visual mesh filename=../meshes/base_link.STL
- link camera_link: geometry collision mesh filename=../meshes/camera_link.STL; visual mesh filename=../meshes/camera_link.STL
- link imu_link: geometry collision mesh filename=../meshes/imu_link.STL; visual mesh filename=../meshes/imu_link.STL
- link left_end_effector_link: geometry collision mesh filename=../meshes/left_end_effector_link.STL; visual mesh filename=../meshes/left_end_effector_link.STL
- link left_foot_pitch_link: geometry collision mesh filename=../meshes/left_foot_pitch_link.STL; visual mesh filename=../meshes/left_foot_pitch_link.STL
- link left_foot_roll_link: geometry collision mesh filename=../meshes/left_foot_roll_link.STL; visual mesh filename=../meshes/left_foot_roll_link.STL
- link left_hand_yaw_link: geometry collision mesh filename=../meshes/left_hand_yaw_link.STL; visual mesh filename=../meshes/left_hand_yaw_link.STL
- link left_lower_arm_pitch_link: geometry collision mesh filename=../meshes/left_lower_arm_pitch_link.STL; visual mesh filename=../meshes/left_lower_arm_pitch_link.STL
- link left_shank_pitch_link: geometry collision mesh filename=../meshes/left_shank_pitch_link.STL; visual mesh filename=../meshes/left_shank_pitch_link.STL
- link left_thigh_pitch_link: geometry collision mesh filename=../meshes/left_thigh_pitch_link.STL; visual mesh filename=../meshes/left_thigh_pitch_link.STL
- link left_thigh_roll_link: geometry collision mesh filename=../meshes/left_thigh_roll_link.STL; visual mesh filename=../meshes/left_thigh_roll_link.STL
- link left_thigh_yaw_link: geometry collision mesh filename=../meshes/left_thigh_yaw_link.STL; visual mesh filename=../meshes/left_thigh_yaw_link.STL
- link left_upper_arm_pitch_link: geometry collision mesh filename=../meshes/left_upper_arm_pitch_link.STL; visual mesh filename=../meshes/left_upper_arm_pitch_link.STL
- link left_upper_arm_roll_link: geometry collision mesh filename=../meshes/left_upper_arm_roll_link.STL; visual mesh filename=../meshes/left_upper_arm_roll_link.STL
- link left_upper_arm_yaw_link: geometry collision mesh filename=../meshes/left_upper_arm_yaw_link.STL; visual mesh filename=../meshes/left_upper_arm_yaw_link.STL
- link right_end_effector_link: geometry collision mesh filename=../meshes/right_end_effector_link.STL; visual mesh filename=../meshes/right_end_effector_link.STL
- link right_foot_pitch_link: geometry collision mesh filename=../meshes/right_foot_pitch_link.STL; visual mesh filename=../meshes/right_foot_pitch_link.STL
- link right_foot_roll_link: geometry collision mesh filename=../meshes/right_foot_roll_link.STL; visual mesh filename=../meshes/right_foot_roll_link.STL
- link right_hand_yaw_link: geometry collision mesh filename=../meshes/right_hand_yaw_link.STL; visual mesh filename=../meshes/right_hand_yaw_link.STL
- link right_lower_arm_pitch_link: geometry collision mesh filename=../meshes/right_lower_arm_pitch_link.STL; visual mesh filename=../meshes/right_lower_arm_pitch_link.STL
- link right_shank_pitch_link: geometry collision mesh filename=../meshes/right_shank_pitch_link.STL; visual mesh filename=../meshes/right_shank_pitch_link.STL
- link right_thigh_pitch_link: geometry collision mesh filename=../meshes/right_thigh_pitch_link.STL; visual mesh filename=../meshes/right_thigh_pitch_link.STL
- link right_thigh_roll_link: geometry collision mesh filename=../meshes/right_thigh_roll_link.STL; visual mesh filename=../meshes/right_thigh_roll_link.STL
- link right_thigh_yaw_link: geometry collision mesh filename=../meshes/right_thigh_yaw_link.STL; visual mesh filename=../meshes/right_thigh_yaw_link.STL
- link right_upper_arm_pitch_link: geometry collision mesh filename=../meshes/right_upper_arm_pitch_link.STL; visual mesh filename=../meshes/right_upper_arm_pitch_link.STL
- link right_upper_arm_roll_link: geometry collision mesh filename=../meshes/right_upper_arm_roll_link.STL; visual mesh filename=../meshes/right_upper_arm_roll_link.STL
- link right_upper_arm_yaw_link: geometry collision mesh filename=../meshes/right_upper_arm_yaw_link.STL; visual mesh filename=../meshes/right_upper_arm_yaw_link.STL
- link torso_link: geometry collision mesh filename=../meshes/torso_link.STL; visual mesh filename=../meshes/torso_link.STL
- link waist_yaw_link: geometry collision mesh filename=../meshes/waist_yaw_link.STL; visual mesh filename=../meshes/waist_yaw_link.STL
Joints:
- joint left_elbow_pitch_joint: limit lower=-1.884 upper=0.088 effort=29.3 velocity=13.927 -> lower=-0.314 upper=1.658 effort=29.3 velocity=13.927; origin xyz=0 0 -0.105 rpy=0 1.57 0 -> xyz=0 0 -0.105 rpy=0 0 0
- joint left_shoulder_roll_joint: limit lower=-0.375 upper=2.592 effort=29.3 velocity=13.927 -> lower=-0.175 upper=2.792 effort=29.3 velocity=13.927; origin xyz=0 0.082 0 rpy=0.2 0 0 -> xyz=0 0.082 0 rpy=0 0 0
- joint left_shoulder_yaw_joint: type fixed -> revolute
- joint left_wrist_yaw_joint: type fixed -> revolute
- joint right_elbow_pitch_joint: limit lower=-1.884 upper=0.088 effort=29.3 velocity=13.927 -> lower=-0.314 upper=1.658 effort=29.3 velocity=13.927; origin xyz=0 0 -0.105 rpy=0 1.57 0 -> xyz=0 0 -0.105 rpy=0 0 0
- joint right_shoulder_roll_joint: limit lower=-2.592 upper=0.375 effort=29.3 velocity=13.927 -> lower=-2.792 upper=0.175 effort=29.3 velocity=13.927; origin xyz=0 -0.082 0 rpy=-0.2 0 0 -> xyz=0 -0.082 0 rpy=0 0 0
- joint right_shoulder_yaw_joint: type fixed -> revolute
- joint right_wrist_yaw_joint: type fixed -> revolute
