Commit message: 添加floating_base节点

File: src/renderer/public/urdf/GRMini1T1_raw_floating_base.urdf (robot description, URDF)
Before this commit: robot GRMini1T1, 30 links, 29 joints
Links:
- removed link world
- added link world_pitch, mass 0.0
- added link world_roll, mass 0.0
- added link world_yaw, mass 0.0
Joints:
- removed joint floating_base_joint
- added joint floating_base_pitch_joint: type revolute, parent world_pitch, child world_yaw, origin xyz=0 0 0 rpy=0 0 0, axis 0 1 0, limit lower=-3.14159 upper=3.14159 effort=59.8 velocity=12.252
- added joint floating_base_roll_joint: type revolute, parent world_roll, child base_link, origin xyz=0 0 0.70 rpy=0 0 0, axis 1 0 0, limit lower=-3.14159 upper=3.14159 effort=59.8 velocity=12.252
- added joint floating_base_yaw_joint: type revolute, parent world_yaw, child world_roll, origin xyz=0 0 0 rpy=0 0 0, axis 0 0 1, limit lower=-3.14159 upper=3.14159 effort=59.8 velocity=12.252
